File: eagle/Ethernet_Mini_Shield_v0.1.brd (EAGLE design)
At the start: 24 x 25.5 mm, 4 parts, among them U1 RJ45

Commit message: Added version 0.2
Parts:
- added SL4: (no value), con-amp-quick:02P
- moved SL3 3.50 mm to (21.0, 16.4)
Connections:
- removed net SIGNAL: SL3.1, U1.7
- new net +5V: SL3.2, U1.3
- new net END: SL4.2, U1.7
- new net START: SL4.1, U1.5
- net GND: now also SL3.1; no longer SL3.2
Routing:
- net START: track 0.00 -> 23.0 mm
- net +5V: track 0.00 -> 21.5 mm
- net SIGNAL: track 17.2 -> 0.00 mm
- net END: track 0.00 -> 16.2 mm
- net GND: track 15.0 -> 13.9 mm
Other:
- board text added: "+5V"
- board text added: "END"
- board text added: "START"
- board text removed: "CNC"
- board text removed: "Ethernet"
- board text removed: "SIG"
