File: eagle/Ethernet_Mini_Shield_v0.1.sch (EAGLE design)
At the start: 4 parts, among them U1 RJ45

Commit message: Added version 0.2
Parts:
- added SL4: (no value), con-amp-quick:M02
Connections:
- removed net SIGNAL: SL3.1, U1.7
- new net +5V: SL3.2, U1.3
- new net END: SL4.2, U1.7
- new net START: SL4.1, U1.5
- net GND: now also SL3.1; no longer SL3.2
Changed lines of the file:
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@@
 <setting verticaltext="up"/>
 </settings>
-<grid distance="1.27" unitdist="mm" unit="mm" style="lines" multiple="1" display="yes" altdistance="0.01" altunitdist="inch" altunit="inch"/>
+<grid distance="0.05" unitdist="inch" unit="inch" style="lines" multiple="1" display="yes" altdistance="0.01" altunitdist="inch" altunit="inch"/>
 <layers>
 <layer number="1" name="Top" color="4" fill="1" visible="no" active="no"/>
@@
 <part name="U1" library="SparkFun" deviceset="RJ45-8" device="PTH" value="RJ45"/>
 <part name="FRAME1" library="frames" deviceset="A4L-LOC" device=""/>
+<part name="SL4" library="con-amp-quick" deviceset="M02" device=""/>
 </parts>
 <sheets>
@@
 <instance part="U1" gate="G$1" x="163.83" y="109.22"/>
 <instance part="FRAME1" gate="G$1" x="0" y="0"/>
+<instance part="SL4" gate="G$1" x="87.63" y="135.89"/>
 </instances>
 <busses>
@@
 </segment>
 <segment>
+<pinref part="SL3" gate="G$1" pin="1"/>
+<wire x1="95.25" y1="116.84" x2="105.41" y2="116.84" width="0.1524" layer="91"/>
+<label x="106.68" y="116.84" size="1.778" layer="95"/>
+</segment>
+</net>
+<net name="END" class="0">
+<segment>
+<pinref part="SL4" gate="G$1" pin="2"/>
+<wire x1="95.25" y1="138.43" x2="105.41" y2="138.43" width="0.1524" layer="91"/>
+<label x="106.68" y="138.43" size="1.778" layer="95"/>
+</segment>
+<segment>
+<pinref part="U1" gate="G$1" pin="7"/>
+<wire x1="151.13" y1="104.14" x2="140.97" y2="104.14" width="0.1524" layer="91"/>
+<label x="130.81" y="104.14" size="1.778" layer="95"/>
+</segment>
+</net>
+<net name="+5V" class="0">
+<segment>
+<pinref part="U1" gate="G$1" pin="3"/>
+<wire x1="151.13" y1="114.3" x2="140.97" y2="114.3" width="0.1524" layer="91"/>
+<label x="130.81" y="114.3" size="1.778" layer="95"/>
+</segment>
+<segment>
 <pinref part="SL3" gate="G$1" pin="2"/>
 <wire x1="95.25" y1="119.38" x2="105.41" y2="119.38" width="0.1524" layer="91"/>
@@
 </segment>
 </net>
-<net name="SIGNAL" class="0">
-<segment>
-<pinref part="SL3" gate="G$1" pin="1"/>
-<wire x1="95.25" y1="116.84" x2="105.41" y2="116.84" width="0.1524" layer="91"/>
-<label x="106.68" y="116.84" size="1.778" layer="95"/>
-</segment>
-<segment>
-<pinref part="U1" gate="G$1" pin="7"/>
-<wire x1="151.13" y1="104.14" x2="140.97" y2="104.14" width="0.1524" layer="91"/>
-<label x="130.81" y="104.14" size="1.778" layer="95"/>
-</segment>
-</net>
+<net name="START" class="0">
+<segment>
+<pinref part="SL4" gate="G$1" pin="1"/>
+<wire x1="95.25" y1="135.89" x2="105.41" y2="135.89" width="0.1524" layer="91"/>
+<label x="106.68" y="135.89" size="1.778" layer="95"/>
+</segment>
+<segment>
+<pinref part="U1" gate="G$1" pin="5"/>
+<wire x1="151.13" y1="109.22" x2="140.97" y2="109.22" width="0.1524" layer="91"/>
+<label x="130.81" y="109.22" size="1.778" layer="95"/>
+</segment>
+</net>
